Commit message: confocal sensor added

File: Assets/PM_Robot/pm_robot_unity_confocal.urdf (robot description, URDF)
Before this commit: robot pm_robot, 98 links, 81 joints
Links:
- link Tool_Schunk_SPT_Holder: mass 0.0172841989183379 -> 0.000106303297474693; geometry collision mesh filename=meshes/Tools/Schunk_Vacuum_Tools/SPT_Toolholder_old/Tool_Sc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; visual mesh filename=meshes/Tools/Schunk_Vacuum_Tools/SPT_Toolholder_old/Tool_Sc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
- link Tool_Tip_R_A1000_I500: mass 0.00106303297474693 -> 0.000106303297474693; geometry collision mesh filename=meshes/Tools/Schunk_Vacuum_Tools/SPT_Toolholder_old/Tips/To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; visual mesh filename=meshes/Tools/Schunk_Vacuum_Tools/SPT_Toolholder_old/Tips/To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
Joints:
- removed joint 1K_Dispenser_Flap_Joint
- added joint 1K_Dispenser_Protection_Joint: type prismatic, parent Z_Axis, child Glue_Cartridge_Flap, origin xyz=-0.0315 -0.02479 -0.424 rpy=0 0 0, axis -1 0 0, limit lower=-0.025 upper=0.00 effort=100 velocity=0.5
- joint Gonio_Left_Chuck_Joint: child Chuck_Siemens_Sensor -> Chuck_ipeg_Demonstrator
- joint Gonio_Left_Part_Origin_Joint: origin xyz=0.0175 0.023 0.09655 rpy=0 0 0 -> xyz=0.01 0.015 0.10105 rpy=0 0 0
- joint Gonio_Right_Part_2_Origin_Joint: origin xyz=0.0 0.0 0.0 rpy=0 0 0 -> xyz=-0.009782273 0.0 0.056053231 rpy=0 0 0
- joint UV_Slider_X_Back_Joint: origin xyz=0.0785000000000389 0.200000000000049 0.234999999999998 rpy=0 0 0 -> xyz=0.1241 0.200000000000049 0.234999999999998 rpy=0 0 0
- joint UV_Slider_X_Front_Joint: origin xyz=0.0785000000000391 0.0200000000000492 0.234999999999997 rpy=0 0 0 -> xyz=0.1241 0.0200000000000492 0.234999999999997 rpy=0 0 0
