Commit message: bug fix left gonio

File: Assets/PM_Robot/pm_robot_unity_p39.urdf (robot description, URDF)
Before this commit: robot pm_robot, 102 links, 81 joints
Links:
- removed link Tool_Holder_Siemens_Vacuum_Array_short
- added link Jaw_Flat_Config_ROS_Jaw1, mass 0.000118476289547731; collision mesh filename=meshes/Tools/Parallel_Gripper_1_Jaw/SmarAct_Piezo_Gripper/J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; visual mesh filename=meshes/Tools/Parallel_Gripper_1_Jaw/SmarAct_Piezo_Gripper/J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
- added link Jaw_Flat_Config_ROS_Jaw2, mass 0.000117826998616915; collision mesh filename=meshes/Tools/Parallel_Gripper_1_Jaw/SmarAct_Piezo_Gripper/J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; visual mesh filename=meshes/Tools/Parallel_Gripper_1_Jaw/SmarAct_Piezo_Gripper/J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
- added link SmarAct_Gripper_Jaw_flat, mass 0.000125699746806344; collision mesh filename=meshes/Tools/Parallel_Gripper_1_Jaw/SmarAct_Piezo_Gripper/S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; visual mesh filename=meshes/Tools/Parallel_Gripper_1_Jaw/SmarAct_Piezo_Gripper/S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
- added link Tool_Parallel_Gripper_Base_flat, mass 0.0122161706567272; collision mesh filename=meshes/Tools/Parallel_Gripper_1_Jaw/SmarAct_Piezo_Gripper/T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; visual mesh filename=meshes/Tools/Parallel_Gripper_1_Jaw/SmarAct_Piezo_Gripper/T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
Joints:
- added joint Tool_Parallel_Gripper_Body_Joint: type fixed, parent t_axis_tool, child Tool_Parallel_Gripper_Base_flat, origin xyz=0 0 -0.04542 rpy=0 0 0, axis 0 0 0
- added joint Tool_Parallel_Gripper_Jaw_1_Point_Joint: type fixed, parent Tool_Parallel_Gripper_Base_flat, child Tool_Parallel_Gripper_Jaw_1_Point, origin xyz=-0.00549999981186566 0.00150000018813442 -0.0318 rpy=0 0 0, axis 0 0 0
- added joint Tool_Parallel_Gripper_Jaw_1_attachment_Joint: type fixed, parent Tool_Parallel_Gripper_Jaw_1_Point, child Jaw_Flat_Config_ROS_Jaw1, origin xyz=0.0 0.0 0  rpy=0 0 0
- added joint Tool_Parallel_Gripper_Jaw_2_Point_Joint: type fixed, parent SmarAct_Gripper_Jaw_flat, child Tool_Parallel_Gripper_Jaw_2_Point, origin xyz=0.0 0 0 rpy=0 0 0, axis 0 0 0
- added joint Tool_Parallel_Gripper_Jaw_2_attachment_Joint: type fixed, parent Tool_Parallel_Gripper_Jaw_2_Point, child Jaw_Flat_Config_ROS_Jaw2, origin xyz=0.0 0 0  rpy=0 0 0
- added joint Tool_Parallel_Gripper_Jaw_Joint: type prismatic, parent Tool_Parallel_Gripper_Base_flat, child SmarAct_Gripper_Jaw_flat, origin xyz=0.00551408822663166 0.00150000018813439 -0.0318 rpy=0 0 0, axis 1 0 0, limit lower=0 upper=0.001 effort=20 velocity=0.05
- joint PM_Robot_Tool_TCP_Joint: child PM_Robot_Tool_TCP_Tip_Lens_12_7_long -> PM_Robot_Tool_TCP; origin xyz=       0.0        0.0        -0.08942 rpy=       0.0        0.0        0.0 -> xyz=       0.0        0.0        -0.08322 rpy=       0.0        0.0        0.0

Commit message: spawning assembly scene

File: Assets/PM_Robot/pm_robot_unity_p39.urdf (robot description, URDF)
Before this commit: robot pm_robot, 105 links, 87 joints
Links:
- added link Default_Jaw_1, mass 0.000118476289547731; collision mesh filename=meshes/Tools/Parallel_Gripper_1_Jaw/SmarAct_Piezo_Gripper/D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; visual mesh filename=meshes/Tools/Parallel_Gripper_1_Jaw/SmarAct_Piezo_Gripper/D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
- added link Default_Jaw_2, mass 0.000117826998616915; collision mesh filename=meshes/Tools/Parallel_Gripper_1_Jaw/SmarAct_Piezo_Gripper/D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; visual mesh filename=meshes/Tools/Parallel_Gripper_1_Jaw/SmarAct_Piezo_Gripper/D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
- added link SmarAct_Gripper_Base, mass 0.0122161706567272; collision mesh filename=meshes/Tools/Parallel_Gripper_1_Jaw/SmarAct_Piezo_Gripper/S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; visual mesh filename=meshes/Tools/Parallel_Gripper_1_Jaw/SmarAct_Piezo_Gripper/S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
- added link SmarAct_Gripper_Jaw, mass 0.000125699746806344; collision mesh filename=meshes/Tools/Parallel_Gripper_1_Jaw/SmarAct_Piezo_Gripper/S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; visual mesh filename=meshes/Tools/Parallel_Gripper_1_Jaw/SmarAct_Piezo_Gripper/S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
- added link Tool_Parallel_Gripper_Jaw_1_Point
- added link Tool_Parallel_Gripper_Jaw_2_Point
