Commit message: bug fix gonio_part_origin

File: Assets/PM_Robot/pm_robot_unity_smarpod.urdf (robot description, URDF)
Before this commit: robot pm_robot, 98 links, 81 joints
Links:
- removed link Tip_Lens_12_7
- removed link Tip_Lens_12_7_long
- removed link Tool_Holder_Siemens_Vacuum_Array
- removed link Tool_Schunk_Lens_Holder
- removed link Tool_Schunk_Lens_Holder_long
- removed link Tool_Schunk_SPT_Holder
- removed link Tool_Tip_R_A1000_I500
- removed link Tool_Tip_Vacuum_Array
- added link Aufnahme_Siemens_SIN, mass 0.0856656121839983; collision mesh filename=meshes/Gonio_Right/Gonio_Right_Chucks/Aufnahme_Siemens_SIN.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; visual mesh filename=meshes/Gonio_Right/Gonio_Right_Chucks/Aufnahme_Siemens_SIN.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
- added link Chuck_Siemens_Carrier_P39, mass 0.122033650525121; collision mesh filename=meshes/Gonio_Left/Gonio_Left_Chucks/Chuck_Siemens_Carrier_P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; visual mesh filename=meshes/Gonio_Left/Gonio_Left_Chucks/Chuck_Siemens_Carrier_P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
- added link Chuck_Siemens_Carrier_SIN, mass 0.193859196068301; collision mesh filename=meshes/Gonio_Left/Gonio_Left_Chucks/Chuck_Siemens_Carrier_S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; visual mesh filename=meshes/Gonio_Left/Gonio_Left_Chucks/Chuck_Siemens_Carrier_S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
- added link Default_Jaw_1, mass 0.000118476289547731; collision mesh filename=meshes/Tools/Parallel_Gripper_1_Jaw/SmarAct_Piezo_Gripper/D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; visual mesh filename=meshes/Tools/Parallel_Gripper_1_Jaw/SmarAct_Piezo_Gripper/D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
- added link Default_Jaw_2, mass 0.000117826998616915; collision mesh filename=meshes/Tools/Parallel_Gripper_1_Jaw/SmarAct_Piezo_Gripper/D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; visual mesh filename=meshes/Tools/Parallel_Gripper_1_Jaw/SmarAct_Piezo_Gripper/D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
- added link Jaw_Flat_Config_ROS_Jaw1, mass 0.000118476289547731; collision mesh filename=meshes/Tools/Parallel_Gripper_1_Jaw/SmarAct_Piezo_Gripper/J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; visual mesh filename=meshes/Tools/Parallel_Gripper_1_Jaw/SmarAct_Piezo_Gripper/J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
- added link Jaw_Flat_Config_ROS_Jaw2, mass 0.000117826998616915; collision mesh filename=meshes/Tools/Parallel_Gripper_1_Jaw/SmarAct_Piezo_Gripper/J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; visual mesh filename=meshes/Tools/Parallel_Gripper_1_Jaw/SmarAct_Piezo_Gripper/J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
- added link SmarAct_Gripper_Base, mass 0.0122161706567272; collision mesh filename=meshes/Tools/Parallel_Gripper_1_Jaw/SmarAct_Piezo_Gripper/S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; visual mesh filename=meshes/Tools/Parallel_Gripper_1_Jaw/SmarAct_Piezo_Gripper/S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
- added link SmarAct_Gripper_Jaw, mass 0.000125699746806344; collision mesh filename=meshes/Tools/Parallel_Gripper_1_Jaw/SmarAct_Piezo_Gripper/S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; visual mesh filename=meshes/Tools/Parallel_Gripper_1_Jaw/SmarAct_Piezo_Gripper/S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
- added link SmarAct_Gripper_Jaw_flat, mass 0.000125699746806344; collision mesh filename=meshes/Tools/Parallel_Gripper_1_Jaw/SmarAct_Piezo_Gripper/S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; visual mesh filename=meshes/Tools/Parallel_Gripper_1_Jaw/SmarAct_Piezo_Gripper/S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
- added link Tool_Parallel_Gripper_Base_flat, mass 0.0122161706567272; collision mesh filename=meshes/Tools/Parallel_Gripper_1_Jaw/SmarAct_Piezo_Gripper/T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; visual mesh filename=meshes/Tools/Parallel_Gripper_1_Jaw/SmarAct_Piezo_Gripper/T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
- added link Tool_Parallel_Gripper_Jaw_1_Point
- added link Tool_Parallel_Gripper_Jaw_2_Point
Joints:
- removed joint 1K_Dispenser_Flap_Joint
- removed joint PM_Robot_Vacuum_Tool_Joint
- removed joint PM_Robot_Vacuum_Tool_Tip_Joint
- added joint 1K_Dispenser_Protection_Joint: type prismatic, parent Z_Axis, child Glue_Cartridge_Flap, origin xyz=-0.0315 -0.02479 -0.424 rpy=0 0 0, axis -1 0 0, limit lower=-0.025 upper=0.00 effort=100 velocity=0.5
- added joint Tool_Parallel_Gripper_Body_Joint: type fixed, parent t_axis_tool, child Tool_Parallel_Gripper_Base_flat, origin xyz=0 0 -0.04542 rpy=0 0 0, axis 0 0 0
- added joint Tool_Parallel_Gripper_Jaw_1_Point_Joint: type fixed, parent Tool_Parallel_Gripper_Base_flat, child Tool_Parallel_Gripper_Jaw_1_Point, origin xyz=-0.00549999981186566 0.00150000018813442 -0.0318 rpy=0 0 0, axis 0 0 0
- added joint Tool_Parallel_Gripper_Jaw_1_attachment_Joint: type fixed, parent Tool_Parallel_Gripper_Jaw_1_Point, child Jaw_Flat_Config_ROS_Jaw1, origin xyz=0.0 0.0 0  rpy=0 0 0
- added joint Tool_Parallel_Gripper_Jaw_2_Point_Joint: type fixed, parent SmarAct_Gripper_Jaw_flat, child Tool_Parallel_Gripper_Jaw_2_Point, origin xyz=0.0 0 0 rpy=0 0 0, axis 0 0 0
- added joint Tool_Parallel_Gripper_Jaw_2_attachment_Joint: type fixed, parent Tool_Parallel_Gripper_Jaw_2_Point, child Jaw_Flat_Config_ROS_Jaw2, origin xyz=0.0 0 0  rpy=0 0 0
- added joint Tool_Parallel_Gripper_Jaw_Joint: type prismatic, parent Tool_Parallel_Gripper_Base_flat, child SmarAct_Gripper_Jaw_flat, origin xyz=0.00551408822663166 0.00150000018813439 -0.0318 rpy=0 0 0, axis 1 0 0, limit lower=0 upper=0.001 effort=20 velocity=0.05
- joint Calibration_Qube_Joint: origin xyz=           0.154            0.108            0.305 rpy=           0.0            0.0            0.0 -> xyz=           0.154            0.108            0.303733 rpy=           0.0            0.0            0.0
- joint Cam1_Toolhead_TCP_Joint: origin xyz=         -0.0320000000000003          -0.0579999999999998          -0.515338706 rpy=         0.0          0.0          0.0 -> xyz=         -0.0320000000000003          -0.0579999999999998          -0.5179414 rpy=         0.0          0.0          0.0
- joint Camera_Station_TCP_Joint: origin xyz=         0.08          0.092783          0.3045 rpy=         0.0          0.0          0.0 -> xyz=         0.08          0.092783          0.2985 rpy=         0.0          0.0          0.0
- joint Gonio_Left_Chuck_Joint: child Chuck_Siemens_Sensor -> Chuck_ipeg_Demonstrator
- joint Gonio_Left_Part_Origin_Joint: origin xyz=0.0175 0.023 0.09655 rpy=0 0 0 -> xyz=0.01 0.015 0.10105 rpy=0 0 0
- joint Gonio_Right_Part_2_Origin_Joint: origin xyz=0.0 0.0 0.0 rpy=0 0 0 -> xyz=-0.009782273 0.0 0.056053231 rpy=0 0 0
- joint PM_Robot_Tool_TCP_Joint: child PM_Robot_Tool_TCP_Tip_Lens_12_7_long -> PM_Robot_Tool_TCP; origin xyz=       0.0        0.0        -0.08942 rpy=       0.0        0.0        0.0 -> xyz=       0.0        0.0        -0.08322 rpy=       0.0        0.0        0.0
- joint SmarPod_Origin_Joint: origin xyz=0 0 0 rpy=0 0 0 -> xyz=0 0 0.00 rpy=0 0 0
- joint Smarpod_Station_Base_Joint: origin xyz=0.09 0.0899999999999999 0.2136999999992 rpy=0 0 0 -> xyz=0.2 0.15 0.2253999999992 rpy=0 0 0
- joint Smarpod_Station_Joint: origin xyz=0.750000000000003 0.315 0 rpy=0 0 0 -> xyz=0.6 0.31 0 rpy=0 0 0
- joint T_Axis_Joint: limit lower=-2.0 upper=2.0 effort=100 velocity=5 -> lower=-2.0 upper=2.0 effort=100 velocity=15; origin xyz=0.0600000000000017 -0.0580000000000003 -0.427500000000004 rpy=0 0 0 -> xyz=         0.0600000000000017          -0.0580000000000003          -0.427500000000004 rpy=         0.0          0.0          0.0
- joint UV_Slider_X_Back_Joint: origin xyz=0.0785000000000389 0.200000000000049 0.234999999999998 rpy=0 0 0 -> xyz=0.1241 0.200000000000049 0.234999999999998 rpy=0 0 0
- joint UV_Slider_X_Front_Joint: origin xyz=0.0785000000000391 0.0200000000000492 0.234999999999997 rpy=0 0 0 -> xyz=0.1241 0.0200000000000492 0.234999999999997 rpy=0 0 0
- joint Z_Axis_Joint: origin xyz=-0.00365 -0.499 0.28525 rpy=0 0 0 -> xyz=-0.00365 -0.499 0.28505 rpy=0 0 0

Commit message: gonio right fix and vacuum_array_short

File: Assets/PM_Robot/pm_robot_unity_smarpod.urdf (robot description, URDF)
Before this commit: robot pm_robot, 103 links, 85 joints
Links:
- removed link Default_Jaw_1
- removed link Default_Jaw_2
- removed link Jaw_Flat_Config_ROS_Jaw1
- removed link Jaw_Flat_Config_ROS_Jaw2
- removed link SmarAct_Gripper_Base
- removed link SmarAct_Gripper_Jaw
- removed link SmarAct_Gripper_Jaw_flat
- removed link Tool_Parallel_Gripper_Base_flat
- removed link Tool_Parallel_Gripper_Jaw_1_Point
- removed link Tool_Parallel_Gripper_Jaw_2_Point
- added link Tip_Lens_12_7, mass 0.00384481220269709; collision mesh filename=meshes/Tools/Schunk_Vacuum_Tools/Lens_Gripper/Tips/Tip_Lens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; visual mesh filename=meshes/Tools/Schunk_Vacuum_Tools/Lens_Gripper/Tips/Tip_Lens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
- added link Tip_Lens_12_7_long, mass 0.00230092030303971; collision mesh filename=meshes/Tools/Schunk_Vacuum_Tools/Lens_Gripper_long/Tips/Tip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; visual mesh filename=meshes/Tools/Schunk_Vacuum_Tools/Lens_Gripper_long/Tips/Tip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
- added link Tool_Holder_Siemens_Vacuum_Array, mass 0.0221301374746933; collision mesh filename=meshes/Tools/Schunk_Vacuum_Tools/Siemens_Vacuum_Array/Tool_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; visual mesh filename=meshes/Tools/Schunk_Vacuum_Tools/Siemens_Vacuum_Array/Tool_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
- added link Tool_Holder_Siemens_Vacuum_Array_short, mass 0.0221301374746933; collision mesh filename=meshes/Tools/Schunk_Vacuum_Tools/Siemens_Vacuum_Array/Tool_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; visual mesh filename=meshes/Tools/Schunk_Vacuum_Tools/Siemens_Vacuum_Array/Tool_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
- added link Tool_Schunk_Lens_Holder, mass 0.000252215142180128; collision mesh filename=meshes/Tools/Schunk_Vacuum_Tools/Lens_Gripper/Tool_Schunk_L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; visual mesh filename=meshes/Tools/Schunk_Vacuum_Tools/Lens_Gripper/Tool_Schunk_L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
- added link Tool_Schunk_Lens_Holder_long, mass 0.0201926555806949; collision mesh filename=meshes/Tools/Schunk_Vacuum_Tools/Lens_Gripper_long/Tool_Sch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; visual mesh filename=meshes/Tools/Schunk_Vacuum_Tools/Lens_Gripper_long/Tool_Sch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
- added link Tool_Schunk_SPT_Holder, mass 0.000106303297474693; collision mesh filename=meshes/Tools/Schunk_Vacuum_Tools/SPT_Toolholder_old/Tool_Sc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; visual mesh filename=meshes/Tools/Schunk_Vacuum_Tools/SPT_Toolholder_old/Tool_Sc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
- added link Tool_Tip_R_A1000_I500, mass 0.000106303297474693; collision mesh filename=meshes/Tools/Schunk_Vacuum_Tools/SPT_Toolholder_old/Tips/To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; visual mesh filename=meshes/Tools/Schunk_Vacuum_Tools/SPT_Toolholder_old/Tips/To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
- added link Tool_Tip_Vacuum_Array, mass 0.00384481220269709; collision mesh filename=meshes/Tools/Schunk_Vacuum_Tools/Siemens_Vacuum_Array/Tool_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; visual mesh filename=meshes/Tools/Schunk_Vacuum_Tools/Siemens_Vacuum_Array/Tool_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
Joints:
- removed joint Tool_Parallel_Gripper_Body_Joint
- removed joint Tool_Parallel_Gripper_Jaw_1_Point_Joint
- removed joint Tool_Parallel_Gripper_Jaw_1_attachment_Joint
- removed joint Tool_Parallel_Gripper_Jaw_2_Point_Joint
- removed joint Tool_Parallel_Gripper_Jaw_2_attachment_Joint
- removed joint Tool_Parallel_Gripper_Jaw_Joint
- added joint PM_Robot_Vacuum_Tool_Joint: type fixed, parent PM_Robot_Tool_TCP, child Tool_Schunk_Lens_Holder_long, origin xyz=0 0 0 rpy=0 0 0, axis 0 0 0
- added joint PM_Robot_Vacuum_Tool_Tip_Joint: type fixed, parent PM_Robot_Tool_TCP, child Tip_Lens_12_7_long, origin xyz=0 0 0 rpy=0 0 0, axis 0 0 0
- joint Gonio_Right_Chuck_Origin_Joint: origin xyz=0 0 -0.0499999999999999 rpy=0 0 0 -> xyz=0 0 -0.05 rpy=0 0 0
- joint Gonio_Right_Stage_1_Joint: axis 0 -1 0 -> 1 0 0; origin xyz=0.0324999999999993 0.0326774999999999 0.11 rpy=0 0 0 -> xyz=0.0325000000000002 0.0324999999999998 0.11 rpy=0 0 0
- joint Gonio_Right_Stage_2_Joint: axis -1 0 0 -> 0 -1 0
- joint PM_Robot_Tool_TCP_Joint: origin xyz=       0.0        0.0        -0.08322 rpy=       0.0        0.0        0.0 -> xyz=       0.0        0.0        -0.08942 rpy=       0.0        0.0        0.0
