Commit message: smaract_gripper

File: Assets/PM_Robot/pm_robot_unity_carrier_demo.urdf (robot description, URDF)
Before this commit: robot pm_robot, 108 links, 85 joints
Links:
- removed link SP_A_Axis
- removed link SP_B_Axis
- removed link SP_C_Axis
- removed link SP_X_Axis
- removed link SP_Y_Axis
- removed link SP_Z_Axis
- removed link SmarPod_Origin
- removed link Smarpod_A_Stage_1
- removed link Smarpod_A_Stage_2
- removed link Smarpod_A_Stage_3
- removed link Smarpod_B_Stage_1
- removed link Smarpod_B_Stage_2
- removed link Smarpod_B_Stage_3
- removed link Smarpod_C_Stage_1
- removed link Smarpod_C_Stage_2
- removed link Smarpod_C_Stage_3
- removed link Smarpod_Part_Spawn
- removed link Smarpod_Station
- removed link Smarpod_Station_Base
- removed link Smarpod_Top_Plate
- removed link Tip_Lens_12_7
- removed link Tip_Lens_12_7_long
- removed link Tool_Holder_Siemens_Vacuum_Array
- removed link Tool_Holder_Siemens_Vacuum_Array_short
- removed link Tool_Schunk_Lens_Holder
- removed link Tool_Schunk_Lens_Holder_long
- removed link Tool_Schunk_SPT_Holder
- removed link Tool_Tip_R_A1000_I500
- removed link Tool_Tip_Vacuum_Array
- removed link Top_Plate_A
- removed link Top_Plate_B
- removed link Top_Plate_C
- added link Default_Jaw_1, mass 0.000118476289547731; collision mesh filename=meshes/Tools/Parallel_Gripper_1_Jaw/SmarAct_Piezo_Gripper/D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; visual mesh filename=meshes/Tools/Parallel_Gripper_1_Jaw/SmarAct_Piezo_Gripper/D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
- added link Default_Jaw_2, mass 0.000117826998616915; collision mesh filename=meshes/Tools/Parallel_Gripper_1_Jaw/SmarAct_Piezo_Gripper/D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; visual mesh filename=meshes/Tools/Parallel_Gripper_1_Jaw/SmarAct_Piezo_Gripper/D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
- added link SmarAct_Gripper_Jaw_flat, mass 0.000125699746806344; collision mesh filename=meshes/Tools/Parallel_Gripper_1_Jaw/SmarAct_Piezo_Gripper/S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; visual mesh filename=meshes/Tools/Parallel_Gripper_1_Jaw/SmarAct_Piezo_Gripper/S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
- added link Tool_Parallel_Gripper_Base_flat, mass 0.0122161706567272; collision mesh filename=meshes/Tools/Parallel_Gripper_1_Jaw/SmarAct_Piezo_Gripper/T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; visual mesh filename=meshes/Tools/Parallel_Gripper_1_Jaw/SmarAct_Piezo_Gripper/T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
- added link Tool_Parallel_Gripper_Jaw_1_Point
- added link Tool_Parallel_Gripper_Jaw_2_Point
Joints:
- removed joint PM_Robot_Vacuum_Tool_Joint
- removed joint PM_Robot_Vacuum_Tool_Tip_Joint
- removed joint SP_A_Joint
- removed joint SP_B_Joint
- removed joint SP_C_Joint
- removed joint SP_X_Joint
- removed joint SP_Y_Joint
- removed joint SP_Z_Joint
- removed joint SmarPod_Origin_Joint
- removed joint Smarpod_A_Stage_1_Joint
- removed joint Smarpod_A_Stage_2_Joint
- removed joint Smarpod_A_Stage_3_Joint
- removed joint Smarpod_B_Stage_1_Joint
- removed joint Smarpod_B_Stage_2_Joint
- removed joint Smarpod_B_Stage_3_Joint
- removed joint Smarpod_C_Stage_1_Joint
- removed joint Smarpod_C_Stage_2_Joint
- removed joint Smarpod_C_Stage_3_Joint
- removed joint Smarpod_Station_Base_Joint
- removed joint Smarpod_Station_Joint
- removed joint Smarpod_Top_Plate_Joint
- removed joint Top_Plate_A_Joint
- removed joint Top_Plate_B_Joint
- removed joint Top_Plate_C_Joint
- removed joint smarpod_part_spawn_joint
- added joint Tool_Parallel_Gripper_Body_Joint: type fixed, parent t_axis_tool, child Tool_Parallel_Gripper_Base_flat, origin xyz=0 0 -0.04542 rpy=0 0 0, axis 0 0 0
- added joint Tool_Parallel_Gripper_Jaw_1_Point_Joint: type fixed, parent Tool_Parallel_Gripper_Base_flat, child Tool_Parallel_Gripper_Jaw_1_Point, origin xyz=-0.00549999981186566 0.00150000018813442 -0.0318 rpy=0 0 0, axis 0 0 0
- added joint Tool_Parallel_Gripper_Jaw_1_attachment_Joint: type fixed, parent Tool_Parallel_Gripper_Jaw_1_Point, child Default_Jaw_1, origin xyz=0.0 0.0 0  rpy=0 0 0
- added joint Tool_Parallel_Gripper_Jaw_2_Point_Joint: type fixed, parent SmarAct_Gripper_Jaw_flat, child Tool_Parallel_Gripper_Jaw_2_Point, origin xyz=0.0 0 0 rpy=0 0 0, axis 0 0 0
- added joint Tool_Parallel_Gripper_Jaw_2_attachment_Joint: type fixed, parent Tool_Parallel_Gripper_Jaw_2_Point, child Default_Jaw_2, origin xyz=0.0 0 0  rpy=0 0 0
- added joint Tool_Parallel_Gripper_Jaw_Joint: type prismatic, parent Tool_Parallel_Gripper_Base_flat, child SmarAct_Gripper_Jaw_flat, origin xyz=-0.0004859117733683402 0.00150000018813439 -0.0318 rpy=0 0 0, axis 1 0 0, limit lower=0 upper=0.001 effort=20 velocity=0.05
- joint Gonio_Base_Right_Joint: origin xyz=         0.7505000000000029          0.911          0.0015 rpy=         0.0          0.0          0.0 -> xyz=         0.7505000000000029          0.311          0.0015 rpy=         0.0          0.0          0.0
- joint PM_Robot_Tool_TCP_Joint: origin xyz=       0.0        0.0        -0.08942 rpy=       0.0        0.0        0.0 -> xyz=       0.0        0.0        -0.04542 rpy=       0.0        0.0        0.0

Commit message: vacuum gripper angled

File: Assets/PM_Robot/pm_robot_unity_carrier_demo.urdf (robot description, URDF)
Before this commit: robot pm_robot, 82 links, 66 joints
Links:
- removed link Default_Jaw_1
- removed link Default_Jaw_2
- removed link SmarAct_Gripper_Jaw_flat
- removed link Tool_Parallel_Gripper_Base_flat
- removed link Tool_Parallel_Gripper_Jaw_1_Point
- removed link Tool_Parallel_Gripper_Jaw_2_Point
- added link Tip_Lens_12_7, mass 0.00384481220269709; collision mesh filename=meshes/Tools/Schunk_Vacuum_Tools/Lens_Gripper/Tips/Tip_Lens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; visual mesh filename=meshes/Tools/Schunk_Vacuum_Tools/Lens_Gripper/Tips/Tip_Lens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
- added link Tip_Lens_12_7_long, mass 0.00230092030303971; collision mesh filename=meshes/Tools/Schunk_Vacuum_Tools/Lens_Gripper_long/Tips/Tip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; visual mesh filename=meshes/Tools/Schunk_Vacuum_Tools/Lens_Gripper_long/Tips/Tip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
- added link Tool_Holder_Siemens_Vacuum_Array, mass 0.0221301374746933; collision mesh filename=meshes/Tools/Schunk_Vacuum_Tools/Siemens_Vacuum_Array/Tool_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; visual mesh filename=meshes/Tools/Schunk_Vacuum_Tools/Siemens_Vacuum_Array/Tool_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
- added link Tool_Holder_Siemens_Vacuum_Array_angled, mass 0.0221301374746933; collision mesh filename=meshes/Tools/Schunk_Vacuum_Tools/Siemens_Vacuum_Array/Tool_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; visual mesh filename=meshes/Tools/Schunk_Vacuum_Tools/Siemens_Vacuum_Array/Tool_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
- added link Tool_Holder_Siemens_Vacuum_Array_short, mass 0.0221301374746933; collision mesh filename=meshes/Tools/Schunk_Vacuum_Tools/Siemens_Vacuum_Array/Tool_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; visual mesh filename=meshes/Tools/Schunk_Vacuum_Tools/Siemens_Vacuum_Array/Tool_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
- added link Tool_Schunk_Lens_Holder, mass 0.000252215142180128; collision mesh filename=meshes/Tools/Schunk_Vacuum_Tools/Lens_Gripper/Tool_Schunk_L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; visual mesh filename=meshes/Tools/Schunk_Vacuum_Tools/Lens_Gripper/Tool_Schunk_L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
- added link Tool_Schunk_Lens_Holder_long, mass 0.0201926555806949; collision mesh filename=meshes/Tools/Schunk_Vacuum_Tools/Lens_Gripper_long/Tool_Sch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; visual mesh filename=meshes/Tools/Schunk_Vacuum_Tools/Lens_Gripper_long/Tool_Sch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
- added link Tool_Schunk_SPT_Holder, mass 0.0172841989183379; collision mesh filename=meshes/Tools/Schunk_Vacuum_Tools/SPT_Toolholder/Tool_Schunk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; visual mesh filename=meshes/Tools/Schunk_Vacuum_Tools/SPT_Toolholder/Tool_Schunk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
- added link Tool_Tip_R_A1000_I500, mass 0.00106303297474693; collision mesh filename=meshes/Tools/Schunk_Vacuum_Tools/SPT_Toolholder/Tips/Tool_T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; visual mesh filename=meshes/Tools/Schunk_Vacuum_Tools/SPT_Toolholder/Tips/Tool_T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
- added link Tool_Tip_Vacuum_Array, mass 0.00384481220269709; collision mesh filename=meshes/Tools/Schunk_Vacuum_Tools/Siemens_Vacuum_Array/Tool_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; visual mesh filename=meshes/Tools/Schunk_Vacuum_Tools/Siemens_Vacuum_Array/Tool_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
Joints:
- removed joint Tool_Parallel_Gripper_Body_Joint
- removed joint Tool_Parallel_Gripper_Jaw_1_Point_Joint
- removed joint Tool_Parallel_Gripper_Jaw_1_attachment_Joint
- removed joint Tool_Parallel_Gripper_Jaw_2_Point_Joint
- removed joint Tool_Parallel_Gripper_Jaw_2_attachment_Joint
- removed joint Tool_Parallel_Gripper_Jaw_Joint
- added joint PM_Robot_Vacuum_Tool_Joint: type fixed, parent PM_Robot_Tool_TCP_Tip_Lens_12_7_long, child Tool_Schunk_Lens_Holder_long, origin xyz=0 0 0 rpy=0 0 0, axis 0 0 0
- added joint PM_Robot_Vacuum_Tool_Tip_Joint: type fixed, parent PM_Robot_Tool_TCP_Tip_Lens_12_7_long, child Tip_Lens_12_7_long, origin xyz=0 0 0 rpy=0 0 0, axis 0 0 0
- joint Gonio_Left_Chuck_Joint: child Chuck_Siemens_Carrier_P39_V2 -> Chuck_Carrier_Demo
- joint Gonio_Left_Part_Origin_Joint: origin xyz=0.0301 0.0 0.069 rpy=0 0 0 -> xyz=0.01 0.015 0.10105 rpy=0 0 0
- joint PM_Robot_Tool_TCP_Joint: origin xyz=       0.0        0.0        -0.04542 rpy=       0.0        0.0        0.0 -> xyz=       0.0        0.0        -0.08942 rpy=       0.0        0.0        0.0

Commit message: sensing jaw

File: Assets/PM_Robot/pm_robot_unity_carrier_demo.urdf (robot description, URDF)
Before this commit: robot pm_robot, 86 links, 62 joints
Links:
- removed link Tip_Lens_12_7
- removed link Tip_Lens_12_7_long
- removed link Tool_Holder_Siemens_Vacuum_Array
- removed link Tool_Holder_Siemens_Vacuum_Array_angled
- removed link Tool_Holder_Siemens_Vacuum_Array_short
- removed link Tool_Schunk_Lens_Holder
- removed link Tool_Schunk_Lens_Holder_long
- removed link Tool_Schunk_SPT_Holder
- removed link Tool_Tip_R_A1000_I500
- removed link Tool_Tip_Vacuum_Array
- added link Jaw_Flat_Config_big_r_ros, mass 0.000117826998616915; collision mesh filename=meshes/Tools/Parallel_Gripper_1_Jaw/SmarAct_Piezo_Gripper/J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; visual mesh filename=meshes/Tools/Parallel_Gripper_1_Jaw/SmarAct_Piezo_Gripper/J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
- added link Jaw_Flat_Config_big_stift_rund_ros, mass 0.000118476289547731; collision mesh filename=meshes/Tools/Parallel_Gripper_1_Jaw/SmarAct_Piezo_Gripper/J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; visual mesh filename=meshes/Tools/Parallel_Gripper_1_Jaw/SmarAct_Piezo_Gripper/J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
- added link SmarAct_Gripper_Jaw_flat, mass 0.000125699746806344; collision mesh filename=meshes/Tools/Parallel_Gripper_1_Jaw/SmarAct_Piezo_Gripper/S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; visual mesh filename=meshes/Tools/Parallel_Gripper_1_Jaw/SmarAct_Piezo_Gripper/S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
- added link Tool_Parallel_Gripper_Base_flat, mass 0.0122161706567272; collision mesh filename=meshes/Tools/Parallel_Gripper_1_Jaw/SmarAct_Piezo_Gripper/T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; visual mesh filename=meshes/Tools/Parallel_Gripper_1_Jaw/SmarAct_Piezo_Gripper/T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
- added link Tool_Parallel_Gripper_Jaw_1_Point
- added link Tool_Parallel_Gripper_Jaw_2_Point
- link 1K_Dispenser: geometry collision mesh filename=meshes/1K_Dispenser_coll.STL; visual mesh filename=meshes/1K_Dispenser.STL
- link 2K_Glue_Cartridge: geometry collision mesh filename=meshes/2K_Glue_Cartridge_Coll.STL; visual mesh filename=meshes/2K_Glue_Cartridge.STL
- link Cam1_Toolhead_TCP: geometry collision mesh filename=meshes/Cam1_Toolhead_TCP_coll.STL; visual mesh filename=meshes/Cam1_Toolhead_TCP.STL
- link Camera_Calibration_Platelet: geometry collision mesh filename=meshes/Camera_Calibration_Platelet_coll.STL; visual mesh filename=meshes/Camera_Calibration_Platelet.STL
- link Camera_Station: geometry collision mesh filename=meshes/Camera_Station_coll.STL; visual mesh filename=meshes/Camera_Station.STL
- link Confocal_Sensor_Top: geometry collision mesh filename=meshes/Confocal_Sensor_Top_coll.STL; visual mesh filename=meshes/Confocal_Sensor_Top.STL
- link Glue_Cartridge_Flap: geometry collision mesh filename=meshes/Glue_Cartridge_Flap_Coll.STL; visual mesh filename=meshes/Glue_Cartridge_Flap.STL
- link Gonio_Base_Right: geometry collision mesh filename=meshes/Gonio_Right/Gonio_Base_Right_Coll.STL; visual mesh filename=meshes/Gonio_Right/Gonio_Base_Right.STL
- link Gonio_Left_Base: geometry collision mesh filename=meshes/Gonio_Left/Gonio_Left_Base_coll.STL; visual mesh filename=meshes/Gonio_Left/Gonio_Left_Base.STL
- link Gripper_Rot_Plate: geometry collision mesh filename=meshes/Gripper_Rot_Plate_coll.STL; visual mesh filename=meshes/Gripper_Rot_Plate.STL
- link UV_Cart_Back: geometry collision mesh filename=meshes/Gonio_Left/UV_Cart_Back_Coll.STL; visual mesh filename=meshes/Gonio_Left/UV_Cart_Back.STL
- link UV_Cart_X_Back: geometry collision mesh filename=meshes/Gonio_Left/UV_Cart_X_Back_Coll.STL; visual mesh filename=meshes/Gonio_Left/UV_Cart_X_Back.STL
- link UV_Cart_X_Front: geometry collision mesh filename=meshes/Gonio_Left/UV_Cart_X_Front_Coll.STL; visual mesh filename=meshes/Gonio_Left/UV_Cart_X_Front.STL
- link X_Axis: geometry collision mesh filename=meshes/X_Axis_coll.STL; visual mesh filename=meshes/X_Axis.STL
- link Y_Axis: geometry collision mesh filename=meshes/Y_Axis_coll.STL; visual mesh filename=meshes/Y_Axis.STL
- link Z_Axis: geometry collision mesh filename=meshes/Z_Axis_coll.STL; visual mesh filename=meshes/Z_Axis.STL
- link axis_base: geometry collision mesh filename=meshes/axis_base_coll.STL; visual mesh filename=meshes/axis_base.STL
- link t_axis_tool: geometry collision mesh filename=meshes/t_axis_tool_coll.STL; visual mesh filename=meshes/t_axis_tool.STL
Joints:
- removed joint PM_Robot_Vacuum_Tool_Joint
- removed joint PM_Robot_Vacuum_Tool_Tip_Joint
- added joint Tool_Parallel_Gripper_Body_Joint: type fixed, parent t_axis_tool, child Tool_Parallel_Gripper_Base_flat, origin xyz=0 0 -0.04542 rpy=0 0 0, axis 0 0 0
- added joint Tool_Parallel_Gripper_Jaw_1_Point_Joint: type fixed, parent Tool_Parallel_Gripper_Base_flat, child Tool_Parallel_Gripper_Jaw_1_Point, origin xyz=-0.00549999981186566 0.00150000018813442 -0.0318 rpy=0 0 0, axis 0 0 0
- added joint Tool_Parallel_Gripper_Jaw_1_attachment_Joint: type fixed, parent Tool_Parallel_Gripper_Jaw_1_Point, child Jaw_Flat_Config_big_stift_rund_ros, origin xyz=0.0 0.0 0  rpy=0 0 0
- added joint Tool_Parallel_Gripper_Jaw_2_Point_Joint: type fixed, parent SmarAct_Gripper_Jaw_flat, child Tool_Parallel_Gripper_Jaw_2_Point, origin xyz=0.0 0 0 rpy=0 0 0, axis 0 0 0
- added joint Tool_Parallel_Gripper_Jaw_2_attachment_Joint: type fixed, parent Tool_Parallel_Gripper_Jaw_2_Point, child Jaw_Flat_Config_big_r_ros, origin xyz=0.0 0 0  rpy=0 0 0
- added joint Tool_Parallel_Gripper_Jaw_Joint: type prismatic, parent Tool_Parallel_Gripper_Base_flat, child SmarAct_Gripper_Jaw_flat, origin xyz=0.01551408822663166 0.00150000018813439 -0.0318 rpy=0 0 0, axis 1 0 0, limit lower=0 upper=0.001 effort=20 velocity=0.05
- joint Gonio_Base_Right_Joint: origin xyz=         0.7505000000000029          0.311          0.0015 rpy=         0.0          0.0          0.0 -> xyz=         0.750000000000003          0.31          0.0 rpy=         0.0          0.0          0.0
- joint PM_Robot_Tool_TCP_Joint: origin xyz=       0.0        0.0        -0.08942 rpy=       0.0        0.0        0.0 -> xyz=       -0.007        -0.005        -0.09142 rpy=       0.0        0.0        0.0
- joint T_Axis_Joint: limit lower=-2.0 upper=2.0 effort=100 velocity=15 -> lower=-2.6179938779916667 upper=3.490658503988889 effort=100 velocity=15
