Commit message: asg chuck

File: Assets/PM_Robot/pm_robot_unity_asg_gripper.urdf (robot description, URDF)
Before this commit: robot pm_robot, 135 links, 103 joints
Links:
- added link PM_Robot_Tool_TCP
- added link PM_Robot_Tool_TCP_Tip_Lens_12_7
- added link PM_Robot_Tool_TCP_Tip_Lens_12_7_long
- added link PM_Robot_Tool_TCP_Tip_R_A1000_I500
- added link PM_Robot_Tool_TCP_Tip_Siemens_Sensor_Bottom
- added link PM_Robot_Tool_TCP_Tip_Siemens_Vacuum_Array
- added link Tip_Lens_12_7, mass 0.00384481220269709; collision mesh filename=meshes/Tools/Schunk_Vacuum_Tools/Lens_Gripper/Tips/Tip_Lens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; visual mesh filename=meshes/Tools/Schunk_Vacuum_Tools/Lens_Gripper/Tips/Tip_Lens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
- added link Tip_Lens_12_7_long, mass 0.00230092030303971; collision mesh filename=meshes/Tools/Schunk_Vacuum_Tools/Lens_Gripper_long/Tips/Tip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; visual mesh filename=meshes/Tools/Schunk_Vacuum_Tools/Lens_Gripper_long/Tips/Tip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
- added link Tip_Siemens_Sensor_Bottom, mass 0.00384481220269709; collision mesh filename=meshes/Tools/Schunk_Vacuum_Tools/Siemens_Vacuum_Array/Tip_S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; visual mesh filename=meshes/Tools/Schunk_Vacuum_Tools/Siemens_Vacuum_Array/Tip_S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
- added link Tool_Holder_Siemens_Vacuum_Array, mass 0.0221301374746933; collision mesh filename=meshes/Tools/Schunk_Vacuum_Tools/Siemens_Vacuum_Array/Tool_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; visual mesh filename=meshes/Tools/Schunk_Vacuum_Tools/Siemens_Vacuum_Array/Tool_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
- added link Tool_Holder_Siemens_Vacuum_Array_angled, mass 0.0221301374746933; collision mesh filename=meshes/Tools/Schunk_Vacuum_Tools/Siemens_Vacuum_Array/Tool_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; visual mesh filename=meshes/Tools/Schunk_Vacuum_Tools/Siemens_Vacuum_Array/Tool_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
- added link Tool_Holder_Siemens_Vacuum_Array_short, mass 0.0221301374746933; collision mesh filename=meshes/Tools/Schunk_Vacuum_Tools/Siemens_Vacuum_Array/Tool_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; visual mesh filename=meshes/Tools/Schunk_Vacuum_Tools/Siemens_Vacuum_Array/Tool_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
- added link Tool_Schunk_Lens_Holder, mass 0.000252215142180128; collision mesh filename=meshes/Tools/Schunk_Vacuum_Tools/Lens_Gripper/Tool_Schunk_L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; visual mesh filename=meshes/Tools/Schunk_Vacuum_Tools/Lens_Gripper/Tool_Schunk_L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
- added link Tool_Schunk_Lens_Holder_long, mass 0.0201926555806949; collision mesh filename=meshes/Tools/Schunk_Vacuum_Tools/Lens_Gripper_long/Tool_Sch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; visual mesh filename=meshes/Tools/Schunk_Vacuum_Tools/Lens_Gripper_long/Tool_Sch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
- added link Tool_Schunk_SPT_Holder, mass 0.000106303297474693; collision mesh filename=meshes/Tools/Schunk_Vacuum_Tools/SPT_Toolholder_old/Tool_Sc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; visual mesh filename=meshes/Tools/Schunk_Vacuum_Tools/SPT_Toolholder_old/Tool_Sc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
- added link Tool_Tip_R_A1000_I500, mass 0.00106303297474693; collision mesh filename=meshes/Tools/Schunk_Vacuum_Tools/SPT_Toolholder/Tips/Tool_T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; visual mesh filename=meshes/Tools/Schunk_Vacuum_Tools/SPT_Toolholder/Tips/Tool_T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
- added link Tool_Tip_Vacuum_Array, mass 0.00384481220269709; collision mesh filename=meshes/Tools/Schunk_Vacuum_Tools/Siemens_Vacuum_Array/Tool_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; visual mesh filename=meshes/Tools/Schunk_Vacuum_Tools/Siemens_Vacuum_Array/Tool_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
Joints:
- added joint PM_Robot_Tool_TCP_Joint: type fixed, parent Gripper_Rot_Plate, child PM_Robot_Tool_TCP_Tip_Lens_12_7_long, origin xyz=       0.0        0.0        -0.08942 rpy=       0.0        0.0        0.0, axis 0 0 0
- added joint PM_Robot_Vacuum_Tool_Joint: type fixed, parent PM_Robot_Tool_TCP_Tip_Lens_12_7_long, child Tool_Schunk_Lens_Holder_long, origin xyz=0 0 0 rpy=0 0 0, axis 0 0 0
- added joint PM_Robot_Vacuum_Tool_Tip_Joint: type fixed, parent PM_Robot_Tool_TCP_Tip_Lens_12_7_long, child Tip_Lens_12_7_long, origin xyz=0 0 0 rpy=0 0 0, axis 0 0 0
- joint Gonio_Left_Part_Origin_Joint: origin xyz=0.0164 0.00859 0.1 rpy=0 0 0 -> xyz=0.0301 0.0 0.069 rpy=0 0 0
