Commit message: smarpod import

File: Assets/PM_Robot/pm_robot_unity.urdf (robot description, URDF)
Before this commit: robot pm_robot, 157 links, 141 joints
Links:
- added link Baugruppe_Smarpod_Chucks_Fiber, mass 0.129863306528145; collision mesh filename=meshes/chucks/Baugruppe_Smarpod_Chucks_Fiber.STL; visual mesh filename=meshes/chucks/Baugruppe_Smarpod_Chucks_Fiber.STL
- added link Chuck_Diodenplacement, mass 0.129863306528145; collision mesh filename=meshes/chucks/Chuck_Diodenplacement.STL; visual mesh filename=meshes/chucks/Chuck_Diodenplacement.STL
- added link Chuck_Smarpod_Calibration_Ball, mass 0.129863306528145; collision mesh filename=meshes/chucks/Chuck_Smarpod_Calibration_Ball.STL; visual mesh filename=meshes/chucks/Chuck_Smarpod_Calibration_Ball.STL
- added link Chuck_center_fiber_chip_alignment, mass 0.129863306528145; collision mesh filename=meshes/chucks_center/Chuck_center_fiber_chip_alignment.STL; visual mesh filename=meshes/chucks_center/Chuck_center_fiber_chip_alignment.STL
- added link SP_A_Axis, mass 3.46651857022574
- added link SP_B_Axis, mass 3.46651857022574
- added link SP_C_Axis, mass 3.46651857022574
- added link SP_X_Axis, mass 3.46651857022574
- added link SP_Y_Axis, mass 3.46651857022574
- added link SP_Z_Axis, mass 3.46651857022574
- added link SmarPod_Origin, mass 500.360244074757092; collision mesh filename=meshes/SmarPod_Origin.STL; visual mesh filename=meshes/SmarPod_Origin.STL
- added link Smarpod_A_Stage_1, mass 0.1; collision mesh filename=meshes/Smarpod_A_Stage_1.STL; visual mesh filename=meshes/Smarpod_A_Stage_1.STL
- added link Smarpod_A_Stage_2, mass 0.1; collision mesh filename=meshes/Smarpod_A_Stage_2.STL; visual mesh filename=meshes/Smarpod_A_Stage_2.STL
- added link Smarpod_A_Stage_3, mass 0.1; collision mesh filename=meshes/Smarpod_A_Stage_3.STL; visual mesh filename=meshes/Smarpod_A_Stage_3.STL
- added link Smarpod_B_Stage_1, mass 0.1; collision mesh filename=meshes/Smarpod_B_Stage_1.STL; visual mesh filename=meshes/Smarpod_B_Stage_1.STL
- added link Smarpod_B_Stage_2, mass 0.1; collision mesh filename=meshes/Smarpod_B_Stage_2.STL; visual mesh filename=meshes/Smarpod_B_Stage_2.STL
- added link Smarpod_B_Stage_3, mass 0.1; collision mesh filename=meshes/Smarpod_B_Stage_3.STL; visual mesh filename=meshes/Smarpod_B_Stage_3.STL
- added link Smarpod_C_Stage_1, mass 0.1; collision mesh filename=meshes/Smarpod_C_Stage_1.STL; visual mesh filename=meshes/Smarpod_C_Stage_1.STL
- added link Smarpod_C_Stage_2, mass 0.1; collision mesh filename=meshes/Smarpod_C_Stage_2.STL; visual mesh filename=meshes/Smarpod_C_Stage_2.STL
- added link Smarpod_C_Stage_3, mass 0.1; collision mesh filename=meshes/Smarpod_C_Stage_3.STL; visual mesh filename=meshes/Smarpod_C_Stage_3.STL
- added link Smarpod_Part_Spawn
- added link Smarpod_Part_Spawn_Center
- added link Smarpod_Part_Spawn_Center__unity_source__chuck_fiber_chip_alignment
- added link Smarpod_Part_Spawn_Center__unity_source__empty
- added link Smarpod_Part_Spawn__unity_source__chuck_diodenplacement
- added link Smarpod_Part_Spawn__unity_source__chuck_fiber
- added link Smarpod_Part_Spawn__unity_source__chuck_smarpod_ball_calibration
- added link Smarpod_Part_Spawn__unity_source__chuck_smarpod_calibration
- added link Smarpod_Part_Spawn__unity_source__empty
- added link Smarpod_Pivot_Base_Origin, mass 500.360244074757092
- added link Smarpod_Station, mass 0.782282249809798; collision mesh filename=meshes/Smarpod_Station.STL; visual mesh filename=meshes/Smarpod_Station.STL
- added link Smarpod_Station_Base
- added link Smarpod_Station_Base_Calibration
- added link Smarpod_Top_Plate, mass 0.1; collision mesh filename=meshes/Smarpod_Top_Plate.STL; visual mesh filename=meshes/Smarpod_Top_Plate.STL
- added link Top_Plate_A, mass 1.0
- added link Top_Plate_B, mass 1.0
- added link Top_Plate_C, mass 1.0
- added link calibration_target_holder, mass 0.129863306528145; collision mesh filename=meshes/chucks/calibration_target_holder.STL; visual mesh filename=meshes/chucks/calibration_target_holder.STL
Joints:
- added joint SP_A_Joint: type revolute, parent SP_B_Axis, child SP_A_Axis, origin xyz=0.0 0.0 0.0 rpy=0 0 0, axis 1 0 0, limit lower=-0.349066 upper=0.349066 effort=0.1 velocity=1
- added joint SP_B_Joint: type revolute, parent SP_C_Axis, child SP_B_Axis, origin xyz=0.0 0.0 0.0 rpy=0 0 0, axis 0 1 0, limit lower=-0.349066 upper=0.349066 effort=0.1 velocity=1
- added joint SP_C_Joint: type revolute, parent SP_Z_Axis, child SP_C_Axis, origin xyz=0.0 0.0 0.0 rpy=0 0 0, axis 0 0 1, limit lower=-0.349066 upper=0.349066 effort=0.1 velocity=1
- added joint SP_X_Joint: type prismatic, parent Smarpod_Pivot_Base_Origin, child SP_X_Axis, origin xyz=0.0 0.0 0.0 rpy=0 0 0, axis 1 0 0, limit lower=-0.01 upper=0.01 effort=0.1 velocity=35
- added joint SP_Y_Joint: type prismatic, parent SP_X_Axis, child SP_Y_Axis, origin xyz=0.0 0.0 0.0 rpy=0 0 0, axis 0 1 0, limit lower=-0.01 upper=0.01 effort=0.1 velocity=1
- added joint SP_Z_Joint: type prismatic, parent SP_Y_Axis, child SP_Z_Axis, origin xyz=0.0 0.0 0.0 rpy=0 0 0, axis 0 0 1, limit lower=-0.01 upper=0.01 effort=0.1 velocity=1
- added joint SmarPod_Origin_Joint: type fixed, parent Smarpod_Station_Base, child SmarPod_Origin, origin xyz=0 0 0.0 rpy=0 0 0, axis 0 0 0
- added joint Smarpod_A_Stage_1_Joint: type prismatic, parent SmarPod_Origin, child Smarpod_A_Stage_1, origin xyz=0 -0.11 0.0233 rpy=0 0 0, axis 0 -1 0, limit lower=-0.02 upper=0.02 effort=0.1 velocity=1
- added joint Smarpod_A_Stage_2_Joint: type prismatic, parent Smarpod_A_Stage_1, child Smarpod_A_Stage_2, origin xyz=-0.03 0.0212386752719503 0.011 rpy=0 0 -1.5707963267949, axis 0 -1 0, limit lower=-0.02 upper=0.02 effort=0.1 velocity=1
- added joint Smarpod_A_Stage_3_Joint: type prismatic, parent Smarpod_A_Stage_2, child Smarpod_A_Stage_3, origin xyz=-0.00253689759876602 0.03 0.0259362157397364 rpy=0 0 1.5707963267949, axis 0 -0.86602540378444 0.499999999999997, limit lower=-0.02 upper=0.02 effort=0.1 velocity=1
- added joint Smarpod_B_Stage_1_Joint: type prismatic, parent SmarPod_Origin, child Smarpod_B_Stage_1, origin xyz=-0.0952627944162879 0.0550000000000004 0.0233 rpy=0 0 -2.09439510239321, axis 0 -1 0, limit lower=-0.02 upper=0.02 effort=0.1 velocity=1
- added joint Smarpod_B_Stage_2_Joint: type prismatic, parent Smarpod_B_Stage_1, child Smarpod_B_Stage_2, origin xyz=-0.03 0.0212386752719502 0.0109999999999993 rpy=0 0 -1.5707963267949, axis 0 -1 0, limit lower=-0.02 upper=0.02 effort=0.1 velocity=1
- added joint Smarpod_B_Stage_3_Joint: type prismatic, parent Smarpod_B_Stage_2, child Smarpod_B_Stage_3, origin xyz=-0.00253689759876589 0.03 0.0259362157397364 rpy=0 0 1.5707963267949, axis 0 -0.866025403784442 0.499999999999994, limit lower=-0.02 upper=0.02 effort=0.1 velocity=1
- added joint Smarpod_C_Stage_1_Joint: type prismatic, parent SmarPod_Origin, child Smarpod_C_Stage_1, origin xyz=0.0952627944162877 0.0550000000000009 0.0233 rpy=0 0 2.09439510239321, axis 0 -1 0, limit lower=-0.02 upper=0.02 effort=0.1 velocity=1
- added joint Smarpod_C_Stage_2_Joint: type prismatic, parent Smarpod_C_Stage_1, child Smarpod_C_Stage_2, origin xyz=-0.0300000000000004 0.0212386752719508 0.0109999999999993 rpy=0 0 -1.5707963267949, axis 0 -1 0, limit lower=-0.02 upper=0.02 effort=0.1 velocity=1
- added joint Smarpod_C_Stage_3_Joint: type prismatic, parent Smarpod_C_Stage_2, child Smarpod_C_Stage_3, origin xyz=-0.00253689759876601 0.0299999999999999 0.0259362157397364 rpy=0 0 1.5707963267949, axis 0 -0.866025403784441 0.499999999999995, limit lower=-0.02 upper=0.02 effort=0.1 velocity=1
- added joint Smarpod_Pivot_Base_Origin_Joint: type fixed, parent SmarPod_Origin, child Smarpod_Pivot_Base_Origin, origin xyz=0.0 0.0 0.0573743036851433 rpy=0 0 0, axis 0 0 0
- added joint Smarpod_Station_Base_Calibration_Joint: type fixed, parent Smarpod_Station, child Smarpod_Station_Base_Calibration, origin xyz=         0.1465          0.1          0.2254 rpy=         0          0          0, axis 0 0 0
- added joint Smarpod_Station_Base_Joint: type fixed, parent Smarpod_Station_Base_Calibration, child Smarpod_Station_Base, origin xyz=         -0.001          0.011          0.001 rpy=         0.0          0.0          0.0, axis 0 0 0
- added joint Smarpod_Station_Joint: type fixed, parent pm_robot_base_link, child Smarpod_Station, origin xyz=0.6 0.31 0 rpy=0 0 0, axis 0 0 0
- added joint Smarpod_Top_Plate_Joint: type fixed, parent SP_A_Axis, child Smarpod_Top_Plate, origin xyz=0 0 0 rpy=0 0 0, axis 0 0 0
- added joint Top_Plate_A_Joint: type fixed, parent Smarpod_Top_Plate, child Top_Plate_A, origin xyz=0 -0.0588334882222388 0 rpy=0 0 0, axis 0 0 0
- added joint Top_Plate_B_Joint: type fixed, parent Smarpod_Top_Plate, child Top_Plate_B, origin xyz=-0.0509512951020539 0.0294167446162847 0 rpy=0 0 0, axis 0 0 0
- added joint Top_Plate_C_Joint: type fixed, parent Smarpod_Top_Plate, child Top_Plate_C, origin xyz=0.0509512956853688 0.0294167436059538 0 rpy=0 0 0, axis 0 0 0
- added joint smarpod_chuck_center_joint: type fixed, parent SmarPod_Origin, child Chuck_center_fiber_chip_alignment, origin xyz=0.0 0.0 0.011 rpy=0.0 0.0 0.0
- added joint smarpod_chuck_joint: type fixed, parent Smarpod_Top_Plate, child Chuck_Smarpod_Calibration_Ball, origin xyz=0.0 0.0 0.01763 rpy=0.0 0.0 0.0
- added joint smarpod_part_spawn_center_joint: type fixed, parent Smarpod_Top_Plate, child Smarpod_Part_Spawn_Center, origin xyz=0.0 0.0 0.0
- added joint smarpod_part_spawn_center_joint_unity_source_chuck_fiber_chip_alignment: type fixed, parent Chuck_center_fiber_chip_alignment, child Smarpod_Part_Spawn_Center__unity_source__chuck_fiber_chip_alignment, origin xyz=0.01 0.0035 0.07225
- added joint smarpod_part_spawn_center_joint_unity_source_empty: type fixed, parent Smarpod_Top_Plate, child Smarpod_Part_Spawn_Center__unity_source__empty, origin xyz=0.0 0.0 0.0
- added joint smarpod_part_spawn_joint: type fixed, parent Smarpod_Top_Plate, child Smarpod_Part_Spawn, origin xyz=0.0 0.0 0.0
- added joint smarpod_part_spawn_joint_unity_source_chuck_diodenplacement: type fixed, parent Chuck_Diodenplacement, child Smarpod_Part_Spawn__unity_source__chuck_diodenplacement, origin xyz=0.0 0.0 0.005
- added joint smarpod_part_spawn_joint_unity_source_chuck_fiber: type fixed, parent Baugruppe_Smarpod_Chucks_Fiber, child Smarpod_Part_Spawn__unity_source__chuck_fiber, origin xyz=0.0 -0.015 0.00851
- added joint smarpod_part_spawn_joint_unity_source_chuck_smarpod_ball_calibration: type fixed, parent Chuck_Smarpod_Calibration_Ball, child Smarpod_Part_Spawn__unity_source__chuck_smarpod_ball_calibration, origin xyz=0.01 -0.01 0.0183
- added joint smarpod_part_spawn_joint_unity_source_chuck_smarpod_calibration: type fixed, parent calibration_target_holder, child Smarpod_Part_Spawn__unity_source__chuck_smarpod_calibration, origin xyz=0.0 0.0 0.0055
- added joint smarpod_part_spawn_joint_unity_source_empty: type fixed, parent Smarpod_Top_Plate, child Smarpod_Part_Spawn__unity_source__empty, origin xyz=0.0 0.0 0.0
- joint Gonio_Left_Chuck_Joint: child Chuck_Carrier_Demo -> Chuck_ASG_Dummy

Commit message: confocal config added & bug fixes

File: Assets/PM_Robot/pm_robot_unity.urdf (robot description, URDF)
Before this commit: robot pm_robot, 195 links, 176 joints
Links:
- removed link Confocal_Sensor_Top
- removed link TCP_Confocal_Sensor_Top_2
- added link distance_sensor_z_10_y_16_x_29, mass 0.0655666647000771; collision mesh filename=meshes/distance_sensors/distance_sensor_z_10_y_16_x_29_col.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; visual mesh filename=meshes/distance_sensors/distance_sensor_z_10_y_16_x_29.STL
- added link distance_sensor_z_20_y_16_x_29, mass 0.0655666647000771; collision mesh filename=meshes/distance_sensors/distance_sensor_z_20_y_16_x_29_col.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; visual mesh filename=meshes/distance_sensors/distance_sensor_z_20_y_16_x_29.STL
- added link distance_sensor_z_5_y_16_x_29, mass 0.0655666647000771; collision mesh filename=meshes/distance_sensors/distance_sensor_z_5_y_16_x_29_col.S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; visual mesh filename=meshes/distance_sensors/distance_sensor_z_5_y_16_x_29.STL
Joints:
- removed joint TCP_Confocal_Sensor_Top_2_Joint
- joint TCP_Confocal_Sensor_Top_Joint: child Confocal_Sensor_Top -> distance_sensor_z_20_y_16_x_29; origin xyz=             0.176999957149375              -0.0580000000000008              -0.500500000000003 rpy=             0.0              0.0              0.0 -> xyz=             0.177             -0.057999999999999996             -0.5155 rpy=             0.0              0.0              0.0
